File: Single to split rail DC power supply.kicad_pcb (KiCad board)
At the start: 2 copper layers, 50 parts, among them J1 Screw_Terminal_01x02, J2 Screw_Terminal_01x02, J3 Screw_Terminal_01x02, J4 Screw_Terminal_01x02, Q1 AO3401A, Q2 AO3401A, U1 TPS5430DDA, U2 TPS65131RGER

Commit message: move pcb layout
Parts:
- moved C1 152.1 mm to (60.1, 76.2), turned to 0 degrees
- moved F1 150.9 mm to (53.1, 78.2), turned to 90 degrees
- moved R1 150.4 mm to (56.4, 77.3), turned to -90 degrees
- moved L1 142.4 mm to (55.4, 84.5), turned to -90 degrees
- moved Q1 140.8 mm to (60.7, 80.7), turned to -90 degrees
- moved R2 139.5 mm to (64.6, 78.3), turned to -90 degrees
- moved C3 139.0 mm to (54.9, 89.0), turned to 180 degrees
- moved C4 135.2 mm to (52.9, 95.9), turned to 0 degrees
- moved U1 134.5 mm to (60.8, 87.0), turned to 90 degrees
- moved C2 131.0 mm to (58.9, 93.0), turned to -90 degrees
- moved R3 128.0 mm to (65.1, 89.2), turned to -90 degrees
- moved D1 125.5 mm to (61.1, 96.5), turned to 0 degrees
- moved R4 123.8 mm to (65.1, 93.5), turned to -90 degrees
- moved R12 114.4 mm to (50.4, 103.6), turned to -90 degrees
- moved D4 110.8 mm to (48.5, 103.6), turned to -90 degrees
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Other:
- board outline added: 78.1 x 40 mm

Commit message: finalize the layout
Parts:
- moved C11 1.68 mm to (89.1, 84.3)
- moved C10 1.56 mm to (81.4, 79.3)
- moved C8 1.56 mm to (83.3, 84.5)
- moved C9 1.56 mm to (81.1, 81.2)
- moved D2 1.56 mm to (74.6, 83.0)
- moved R6 1.56 mm to (80.0, 83.2)
- moved R7 1.56 mm to (80.9, 85.2)
- moved R8 1.56 mm to (81.4, 77.2)
- moved C14 1.20 mm to (87.0, 87.1)
- moved C13 1.09 mm to (87.8, 89.2)
- moved L3 0.84 mm to (91.0, 89.5)
- moved R5 0.81 mm to (79.8, 93.8), turned to 180 degrees
- moved C12 0.54 mm to (87.0, 91.2), turned to -90 degrees
- moved H4 0.20 mm to (38.6, 78.4)
- moved H3 0.14 mm to (38.6, 107.2)
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Routing:
- net GND: track 0.00 -> 268.7 mm, vias 0 -> 37
- net +12V: track 0.00 -> 88.6 mm, vias 0 -> 2
- net +5V: track 0.00 -> 84.8 mm, vias 0 -> 4
- net -12V: track 0.00 -> 46.7 mm, vias 0 -> 2
- net Net-(U1-EN): track 0.00 -> 24.1 mm
- net Net-(Q1-S): track 0.00 -> 18.6 mm
- net VCC: track 0.00 -> 17.8 mm
- net Net-(U2-ENN): track 0.00 -> 15.9 mm
- net Net-(D2-A): track 0.00 -> 14.1 mm
- net Net-(Q2-S): track 0.00 -> 13.1 mm, vias 0 -> 2
- net Net-(D3-K): track 0.00 -> 11.5 mm, vias 0 -> 2
- net Net-(Q1-D): track 0.00 -> 11.4 mm
- net Net-(U2-VREF): track 0.00 -> 11.3 mm, vias 0 -> 2
- net Net-(U2-FBP): track 0.00 -> 7.78 mm
- net Net-(U2-FBN): track 0.00 -> 7.42 mm
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- added copper zone on B.Cu, net GND
- added copper zone on F.Cu, net GND
Other:
- board size 78.1 x 40 mm -> 78 x 39.8 mm
- board text added: "+"
- board text added: "+12V"
- board text added: "+5V"
- board text added: "-12V"
- board text added: "GND"
- board text added: "VCC"
